File: Hardware/power.kicad_sch (KiCad schematic)
At the start: 21 parts, among them U3 LM66200DRLR, U4 MAX77827AEFD+T, U5 SC4215

Commit message: PCB Done
Parts:
- TP4, TP5, TP6, TP7, TP8: footprint TestPoint:TestPoint_Pad_D1.5mm -> TestPoint:TestPoint_Pad_D1.0mm
Changed lines of the file:
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@@
       (effects (font (size 1.27 1.27)) (justify left))
     )
-    (property "Footprint" "TestPoint:TestPoint_Pad_D1.5mm" (at 196.85 50.8 0)
+    (property "Footprint" "TestPoint:TestPoint_Pad_D1.0mm" (at 196.85 50.8 0)
       (effects (font (size 1.27 1.27)) hide)
     )
@@
       (effects (font (size 1.27 1.27)) (justify left))
     )
-    (property "Footprint" "TestPoint:TestPoint_Pad_D1.5mm" (at 147.32 34.29 0)
+    (property "Footprint" "TestPoint:TestPoint_Pad_D1.0mm" (at 147.32 34.29 0)
       (effects (font (size 1.27 1.27)) hide)
     )
@@
       (effects (font (size 1.27 1.27)) (justify left))
     )
-    (property "Footprint" "TestPoint:TestPoint_Pad_D1.5mm" (at 128.27 52.07 0)
+    (property "Footprint" "TestPoint:TestPoint_Pad_D1.0mm" (at 128.27 52.07 0)
       (effects (font (size 1.27 1.27)) hide)
     )
@@
       (effects (font (size 1.27 1.27)) (justify left))
     )
-    (property "Footprint" "TestPoint:TestPoint_Pad_D1.5mm" (at 186.69 40.64 0)
+    (property "Footprint" "TestPoint:TestPoint_Pad_D1.0mm" (at 186.69 40.64 0)
       (effects (font (size 1.27 1.27)) hide)
     )
@@
       (effects (font (size 1.27 1.27)))
     )
-    (property "Footprint" "TestPoint:TestPoint_Pad_D1.5mm" (at 161.29 24.13 0)
-      (effects (font (size 1.27 1.27)) hide)
-    )
+    (property "Footprint" "TestPoint:TestPoint_Pad_D1.0mm" (at 161.29 24.13 0)
+      (effects (font (size 1.27 1.27)) hide)
+    )
