File: Hardware/pressure-sensor.kicad_sch (KiCad schematic)
At the start: 15 parts, among them U10 MPRLS0025PA00001A, U6 MPRLS0025PA00001A, U7 MPRLS0025PA00001A, U8 MPRLS0025PA00001A, U9 MPRLS0025PA00001A

Commit message: PCB Done
Parts:
- C18, C19, C28, C29, C30, C31, C32, C33, C34, C35: footprint (none) -> Capacitor_SMD:C_0402_1005Metric
- U10, U6, U7, U8, U9: footprint XDCR_MPRLS0025PA00001A -> PressureSensor:XDCR_MPRLS0025PA00001A
Changed lines of the file:
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@@
       (effects (font (size 1.27 1.27)) (justify left))
     )
-    (property "Footprint" "" (at 88.5952 120.65 0)
+    (property "Footprint" "Capacitor_SMD:C_0402_1005Metric" (at 88.5952 120.65 0)
       (effects (font (size 1.27 1.27)) hide)
     )
@@
       (effects (font (size 1.27 1.27)) (justify left))
     )
-    (property "Footprint" "" (at 87.3252 97.79 0)
+    (property "Footprint" "Capacitor_SMD:C_0402_1005Metric" (at 87.3252 97.79 0)
       (effects (font (size 1.27 1.27)) hide)
     )
@@
       (effects (font (size 1.27 1.27)) (justify left))
     )
-    (property "Footprint" "" (at 84.7852 34.29 0)
+    (property "Footprint" "Capacitor_SMD:C_0402_1005Metric" (at 84.7852 34.29 0)
       (effects (font (size 1.27 1.27)) hide)
     )
@@
       (effects (font (size 1.27 1.27)))
     )
-    (property "Footprint" "XDCR_MPRLS0025PA00001A" (at 58.42 100.33 0)
+    (property "Footprint" "PressureSensor:XDCR_MPRLS0025PA00001A" (at 58.42 100.33 0)
       (effects (font (size 1.27 1.27)) (justify bottom) hide)
     )
@@
       (effects (font (size 1.27 1.27)))
     )
-    (property "Footprint" "XDCR_MPRLS0025PA00001A" (at 59.69 57.15 0)
+    (property "Footprint" "PressureSensor:XDCR_MPRLS0025PA00001A" (at 59.69 57.15 0)
       (effects (font (size 1.27 1.27)) (justify bottom) hide)
     )
@@
       (effects (font (size 1.27 1.27)) (justify left))
     )
-    (property "Footprint" "" (at 88.5952 77.47 0)
+    (property "Footprint" "Capacitor_SMD:C_0402_1005Metric" (at 88.5952 77.47 0)
       (effects (font (size 1.27 1.27)) hide)
     )
@@
       (effects (font (size 1.27 1.27)) (justify left))
     )
-    (property "Footprint" "" (at 158.4452 99.06 0)
+    (property "Footprint" "Capacitor_SMD:C_0402_1005Metric" (at 158.4452 99.06 0)
       (effects (font (size 1.27 1.27)) hide)
     )
@@
       (effects (font (size 1.27 1.27)) (justify left))
     )
-    (property "Footprint" "" (at 159.7152 78.74 0)
+    (property "Footprint" "Capacitor_SMD:C_0402_1005Metric" (at 159.7152 78.74 0)
       (effects (font (size 1.27 1.27)) hide)
     )
@@
       (effects (font (size 1.27 1.27)))
     )
-    (property "Footprint" "XDCR_MPRLS0025PA00001A" (at 129.54 58.42 0)
+    (property "Footprint" "PressureSensor:XDCR_MPRLS0025PA00001A" (at 129.54 58.42 0)
       (effects (font (size 1.27 1.27)) (justify bottom) hide)
     )
@@
       (effects (font (size 1.27 1.27)) (justify left))
     )
-    (property "Footprint" "" (at 87.3252 140.97 0)
+    (property "Footprint" "Capacitor_SMD:C_0402_1005Metric" (at 87.3252 140.97 0)
       (effects (font (size 1.27 1.27)) hide)
     )
@@
       (effects (font (size 1.27 1.27)))
     )
-    (property "Footprint" "XDCR_MPRLS0025PA00001A" (at 129.54 101.6 0)
+    (property "Footprint" "PressureSensor:XDCR_MPRLS0025PA00001A" (at 129.54 101.6 0)
       (effects (font (size 1.27 1.27)) (justify bottom) hide)
     )
@@
       (effects (font (size 1.27 1.27)) (justify left))
     )
-    (property "Footprint" "" (at 159.7152 35.56 0)
+    (property "Footprint" "Capacitor_SMD:C_0402_1005Metric" (at 159.7152 35.56 0)
       (effects (font (size 1.27 1.27)) hide)
     )
@@
       (effects (font (size 1.27 1.27)))
     )
-    (property "Footprint" "XDCR_MPRLS0025PA00001A" (at 58.42 143.51 0)
+    (property "Footprint" "PressureSensor:XDCR_MPRLS0025PA00001A" (at 58.42 143.51 0)
       (effects (font (size 1.27 1.27)) (justify bottom) hide)
     )
@@
       (effects (font (size 1.27 1.27)) (justify left))
     )
-    (property "Footprint" "" (at 158.4452 55.88 0)
+    (property "Footprint" "Capacitor_SMD:C_0402_1005Metric" (at 158.4452 55.88 0)
       (effects (font (size 1.27 1.27)) hide)
     )
@@
       (effects (font (size 1.27 1.27)) (justify left))
     )
-    (property "Footprint" "" (at 88.5952 54.61 0)
-      (effects (font (size 1.27 1.27)) hide)
-    )
+    (property "Footprint" "Capacitor_SMD:C_0402_1005Metric" (at 88.5952 54.61 0)
+      (effects (font (size 1.27 1.27)) hide)
+    )

Commit message: Review Changes Made (except for meme)
Parts:
- C18, C19, C28, C29, C30: value 0.1n -> 0.1u
- C31, C32, C33, C34, C35: value 0.1n -> 1n
Connections:
- net RES: now reaches U7.9 (RES)
- net RES: now also U10.9 (RES), U6.9 (RES), U8.9 (RES), U9.9 (RES)
- no-connect marks 10 -> 5
Changed lines of the file:
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@@
   (no_connect (at 78.74 140.97))
   (no_connect (at 80.01 54.61))
-  (no_connect (at 109.22 55.88))
   (no_connect (at 149.86 99.06))
-  (no_connect (at 38.1 97.79))
-  (no_connect (at 38.1 140.97))
-  (no_connect (at 109.22 99.06))
   (no_connect (at 149.86 55.88))
-  (no_connect (at 39.37 54.61))
   (wire (pts (xy 99.06 109.22) (xy 109.22 109.22))
     (stroke (width 0) (type default))
@@
     (stroke (width 0) (type default))
   )
+  (wire (pts (xy 29.21 54.61) (xy 39.37 54.61))
+    (stroke (width 0) (type default))
+  )
   (wire (pts (xy 83.82 68.58) (xy 83.82 85.09))
     (stroke (width 0) (type default))
@@
     (stroke (width 0) (type default))
   )
+  (wire (pts (xy 99.06 99.06) (xy 109.22 99.06))
+    (stroke (width 0) (type default))
+  )
   (wire (pts (xy 99.06 106.68) (xy 109.22 106.68))
     (stroke (width 0) (type default))
@@
     (stroke (width 0) (type default))
   )
+  (wire (pts (xy 27.94 97.79) (xy 38.1 97.79))
+    (stroke (width 0) (type default))
+  )
   (wire (pts (xy 83.82 111.76) (xy 83.82 128.27))
     (stroke (width 0) (type default))
@@
     (stroke (width 0) (type default))
   )
+  (wire (pts (xy 99.06 55.88) (xy 109.22 55.88))
+    (stroke (width 0) (type default))
+  )
   (wire (pts (xy 153.67 55.88) (xy 157.48 55.88))
     (stroke (width 0) (type default))
@@
     (stroke (width 0) (type default))
   )
+  (wire (pts (xy 25.4 33.02) (xy 21.59 33.02))
+    (stroke (width 0) (type default))
+  )
   (wire (pts (xy 78.74 133.35) (xy 86.36 133.35))
     (stroke (width 0) (type default))
@@
     (stroke (width 0) (type default))
   )
+  (wire (pts (xy 27.94 140.97) (xy 38.1 140.97))
+    (stroke (width 0) (type default))
+  )
   (label "MOSI" (at 99.06 109.22 0) (fields_autoplaced)
     (effects (font (size 1.27 1.27)) (justify left bottom))
   )
+  (label "RES" (at 25.4 33.02 0) (fields_autoplaced)
+    (effects (font (size 1.27 1.27)) (justify left bottom))
+  )
   (label "MOSI" (at 29.21 64.77 0) (fields_autoplaced)
     (effects (font (size 1.27 1.27)) (justify left bottom))
@@
     (effects (font (size 1.27 1.27)) (justify left bottom))
   )
+  (label "RES" (at 99.06 55.88 0) (fields_autoplaced)
+    (effects (font (size 1.27 1.27)) (justify left bottom))
+  )
   (label "MISO" (at 27.94 153.67 0) (fields_autoplaced)
     (effects (font (size 1.27 1.27)) (justify left bottom))
   )
+  (label "RES" (at 27.94 140.97 0) (fields_autoplaced)
+    (effects (font (size 1.27 1.27)) (justify left bottom))
+  )
+  (label "RES" (at 99.06 99.06 0) (fields_autoplaced)
+    (effects (font (size 1.27 1.27)) (justify left bottom))
+  )
+  (label "RES" (at 27.94 97.79 0) (fields_autoplaced)
+    (effects (font (size 1.27 1.27)) (justify left bottom))
+  )
   (label "SCLK" (at 27.94 105.41 0) (fields_autoplaced)
     (effects (font (size 1.27 1.27)) (justify left bottom))
@@
   )
   (label "SCLK" (at 99.06 63.5 0) (fields_autoplaced)
+    (effects (font (size 1.27 1.27)) (justify left bottom))
+  )
+  (label "RES" (at 29.21 54.61 0) (fields_autoplaced)
     (effects (font (size 1.27 1.27)) (justify left bottom))
   )
@@
     (effects (font (size 1.27 1.27)) (justify right))
   )
+  (hierarchical_label "RES" (shape input) (at 21.59 33.02 180) (fields_autoplaced)
+    (effects (font (size 1.27 1.27)) (justify right))
+  )
   (hierarchical_label "SS1" (shape input) (at 39.37 59.69 180) (fields_autoplaced)
     (effects (font (size 1.27 1.27)) (justify right))
@@
       (effects (font (size 1.27 1.27)) (justify left))
     )
-    (property "Value" "0.1n" (at 91.44 118.11 0)
+    (property "Value" "0.1u" (at 91.44 118.11 0)
       (effects (font (size 1.27 1.27)) (justify left))
     )
@@
       (effects (font (size 1.27 1.27)) (justify left))
     )
-    (property "Value" "0.1n" (at 90.17 95.25 0)
+    (property "Value" "1n" (at 90.17 95.25 0)
       (effects (font (size 1.27 1.27)) (justify left))
     )
@@
       (effects (font (size 1.27 1.27)) (justify left))
     )
-    (property "Value" "0.1n" (at 87.63 31.75 0)
+    (property "Value" "0.1u" (at 87.63 31.75 0)
       (effects (font (size 1.27 1.27)) (justify left))
     )
@@
       (effects (font (size 1.27 1.27)) (justify left))
     )
-    (property "Value" "0.1n" (at 91.44 74.93 0)
+    (property "Value" "0.1u" (at 91.44 74.93 0)
       (effects (font (size 1.27 1.27)) (justify left))
     )
@@
       (effects (font (size 1.27 1.27)) (justify left))
     )
-    (property "Value" "0.1n" (at 161.29 96.52 0)
+    (property "Value" "1n" (at 161.29 96.52 0)
       (effects (font (size 1.27 1.27)) (justify left))
     )
@@
       (effects (font (size 1.27 1.27)) (justify left))
     )
-    (property "Value" "0.1n" (at 162.56 76.2 0)
+    (property "Value" "0.1u" (at 162.56 76.2 0)
       (effects (font (size 1.27 1.27)) (justify left))
     )
@@
       (effects (font (size 1.27 1.27)) (justify left))
     )
-    (property "Value" "0.1n" (at 90.17 138.43 0)
+    (property "Value" "1n" (at 90.17 138.43 0)
       (effects (font (size 1.27 1.27)) (justify left))
     )
@@
       (effects (font (size 1.27 1.27)) (justify left))
     )
-    (property "Value" "0.1n" (at 162.56 33.02 0)
+    (property "Value" "0.1u" (at 162.56 33.02 0)
       (effects (font (size 1.27 1.27)) (justify left))
     )
@@
       (effects (font (size 1.27 1.27)) (justify left))
     )
-    (property "Value" "0.1n" (at 161.29 53.34 0)
+    (property "Value" "1n" (at 161.29 53.34 0)
       (effects (font (size 1.27 1.27)) (justify left))
     )
@@
       (effects (font (size 1.27 1.27)) (justify left))
     )
-    (property "Value" "0.1n" (at 91.44 52.07 0)
-      (effects (font (size 1.27 1.27)) (justify left))
-    )
+    (property "Value" "1n" (at 91.44 52.07 0)
+      (effects (font (size 1.27 1.27)) (justify left))
+    )
