File: Hardware/PETE.kicad_pcb (KiCad board)
At the start: 4 copper layers, 61 x 37 mm, 106 parts, among them J1 RBUS, J2 USB_C_Receptacle_USB2.0, J3 Micro_SD_Card_Det, U1 ESP32-S3, U10 MPRLS0025PA00001A, U11 DPS310, U2 SN65HVD230, U3 LM66200DRLR, U4 MAX77827AEFD+T, U5 SC4215, U6 MPRLS0025PA00001A, U7 MPRLS0025PA00001A, U8 MPRLS0025PA00001A, U9 MPRLS0025PA00001A, Y1 40MHz±10ppm

Commit message: artem review
Parts:
- removed BOOT, EN: Conn_01x02_Male, Connector_PinHeader_2.54mm:PinHeader_1x02_P2.54mm_Vertical
- removed the G*** at (69.2, 38.1)
- added 12VLED1: 12V_LED, Resistor_SMD:R_0402_1005Metric, F.Cu at (69.5, 47.5)
- added BOOTJUMPER1: Conn_01x02_Male, Connector_PinHeader_2.54mm:PinHeader_1x02_P2.54mm_Vertical, F.Cu at (71.6, 20.9)
- added ENJUMPER1: Conn_01x02_Male, Connector_PinHeader_2.54mm:PinHeader_1x02_P2.54mm_Vertical, F.Cu at (65.5, 20.9)
- added G***: LOGO, iclr:astronautPete30mmwide, B.Cu at (65.6, 31.9)
- added G***: LOGO, iclr:iclr_logo_estd2018_10mm, B.Cu at (96.5, 45.3)
- added R7: 3k, Resistor_SMD:R_0402_1005Metric, F.Cu at (69.5, 48.5)
- moved C37 3.60 mm to (71.5, 45.8)
- moved TP6 2.87 mm to (51.9, 25.1)
- moved TP8 2.47 mm to (52.3, 37.5)
- moved C36 2.16 mm to (71.9, 44.4), turned to 0 degrees
- moved TP5 1.84 mm to (64.2, 32.8)
- moved U11 1.29 mm to (69.7, 45.1), turned to 180 degrees
- moved R2 1.17 mm to (72.1, 27.0)
- moved TXLED1 1.14 mm to (74.0, 27.0)
- moved TP1 1.11 mm to (69.5, 51.2)
- moved R1 1.00 mm to (65.3, 23.2), turned to 180 degrees
- moved TP2 0.91 mm to (69.5, 54.0)
- moved C17 0.71 mm to (51.0, 41.3)
- moved C8 0.25 mm to (70.3, 23.2)
- moved C3 0.22 mm to (63.5, 23.2)
- moved D1 0.22 mm to (48.6, 41.3)
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Connections:
- U1 pad 16: /MOSI -> /SCLK
- U1 pad 17: /SCLK -> /MOSI
Routing:
- net +3.3V: track 49.1 -> 41.9 mm, vias 17 -> 16
- net GND: track 12.8 -> 7.37 mm, vias 71 -> 70
- net +12V: track 0.00 -> 4.61 mm
- net VBUS: track 46.9 -> 42.9 mm
- net /BARO_CS: track 1.58 -> 5.46 mm
- net /SCLK: track 68.7 -> 72.4 mm
- net /CHIP_PU: track 27.2 -> 24.2 mm
- net /SS4: track 35.0 -> 32.8 mm
- net /Power/BBOUT: track 14.2 -> 12.3 mm
- net /SS5: track 39.4 -> 37.9 mm
- net /MISO: track 66.7 -> 68.1 mm
- net /SS2: track 39.2 -> 37.9 mm
- net /TXD: track 8.57 -> 9.78 mm
- net /SD1_CS: track 15.4 -> 14.2 mm
- net RBUS_uC_V: track 28.0 -> 26.9 mm
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Other:
- board text added: "12V"
- board text added: "BOOT"
- board text added: "Designed by Advay Prabhu Electronics & Payload 2023"
- board text added: "EN"
- board text removed: "Designed by Advay Prabhu!"

Commit message: forgot name of board + some missed drc
Parts:
- moved G*** 1.03 mm to (95.5, 45.3)
- moved TP17 0.39 mm to (81.9, 49.0)
Routing:
- net GND: vias 70 -> 69
Other:
- board text added: "Pete v2.0"

Commit message: ordering
Parts:
- 12VLED1: value 12V_LED -> RED_LED
- 3V3LED1: value 3V3LED -> BLUE_LED
- C12: value 4.2pF -> DNP
- C13, C14: value C -> 11pF
- R13: value 470 -> 5.1k
- R5: value 47.5 -> DNP
- TXLED1: value TX_LED -> GREEN_LED
- USBLED1: value USB_LED -> WHITE_LED
Changed lines of the file:
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@@
         (effects (font (size 0.64 0.64) (thickness 0.16) bold))
     )
-    (fp_text value "TX_LED" (at 0 1.17) (layer "F.Fab")
+    (fp_text value "GREEN_LED" (at 0 1.17) (layer "F.Fab")
         (effects (font (size 1 1) (thickness 0.15)))
     )
@@
         (effects (font (size 1 1) (thickness 0.15)))
     )
-    (fp_text value "C" (at 0 1.16 90) (layer "F.Fab")
+    (fp_text value "11pF" (at 0 1.16 90) (layer "F.Fab")
         (effects (font (size 1 1) (thickness 0.15)))
     )
@@
         (effects (font (size 1 1) (thickness 0.15)))
     )
-    (fp_text value "C" (at 0 1.16 90) (layer "F.Fab")
+    (fp_text value "11pF" (at 0 1.16 90) (layer "F.Fab")
         (effects (font (size 1 1) (thickness 0.15)))
     )
@@
     (fp_line (start 11.1 7.35) (end 11.1 -2.25)
       (stroke (width 0.1) (type solid)) (layer "F.Fab"))
-    (pad "1" thru_hole roundrect (at 0 0 180) (size 2.7 3.3) (drill 1.4) (layers "*.Cu" "*.Mask") (roundrect_rratio 0.092593)
+    (pad "1" thru_hole roundrect (at 0 0 180) (size 2.7 3.3) (drill 1.4) (layers "*.Cu" "*.Mask") (roundrect_rratio 0.09259296296)
       (net 1 "GND") (pinfunction "Pin_1") (pintype "passive"))
     (pad "2" thru_hole oval (at 4.2 0 180) (size 2.7 3.3) (drill 1.4) (layers "*.Cu" "*.Mask")
@@
         (effects (font (size 0.64 0.64) (thickness 0.16)))
     )
-    (fp_text value "3V3LED" (at 0 1.17 90) (layer "F.Fab")
+    (fp_text value "BLUE_LED" (at 0 1.17 90) (layer "F.Fab")
         (effects (font (size 1 1) (thickness 0.15)))
     )
@@
         (effects (font (size 0.635 0.635) (thickness 0.15875) bold))
     )
-    (fp_text value "USB_LED" (at 0 1.17 90) (layer "F.Fab")
+    (fp_text value "WHITE_LED" (at 0 1.17 90) (layer "F.Fab")
         (effects (font (size 1 1) (thickness 0.15)))
     )
@@
         (effects (font (size 1 1) (thickness 0.15)))
     )
-    (fp_text value "4.2pF" (at 0 1.16) (layer "F.Fab")
+    (fp_text value "DNP" (at 0 1.16) (layer "F.Fab")
         (effects (font (size 1 1) (thickness 0.15)))
     )
@@
         (effects (font (size 1 1) (thickness 0.15)))
     )
-    (fp_text value "470" (at 0 1.17 90) (layer "F.Fab")
+    (fp_text value "5.1k" (at 0 1.17 90) (layer "F.Fab")
         (effects (font (size 1 1) (thickness 0.15)))
     )
@@
         (effects (font (size 1 1) (thickness 0.15)))
     )
-    (fp_text value "12V_LED" (at 0 1.17) (layer "F.Fab")
+    (fp_text value "RED_LED" (at 0 1.17) (layer "F.Fab")
         (effects (font (size 1 1) (thickness 0.15)))
     )
@@
         (effects (font (size 1 1) (thickness 0.15)))
     )
-    (fp_text value "47.5" (at 0 1.17) (layer "F.Fab")
+    (fp_text value "DNP" (at 0 1.17) (layer "F.Fab")
         (effects (font (size 1 1) (thickness 0.15)))
     )
