File: Hardware/PETE.kicad_sch (KiCad schematic)
At the start: 54 parts, among them J1 RBUS, J3 Micro_SD_Card_Det, U1 ESP32-S3, U11 DPS310, Y1 40MHz±10ppm

Commit message: PCB Done
Parts:
- TP11, TP12, TP13, TP14, TP15, TP16, TP17, TP18, TP19, TP20, TP21, TP3: footprint (none) -> TestPoint:TestPoint_Pad_D1.0mm
- U1: footprint Package_DFN_QFN:QFN-56-1EP_7x7mm_P0.4mm_EP5.6x5.6mm -> iclr:QFN40P700X700X90-57N
Connections:
- net BARO_CS: now also U1.15 (GPIO10/ADC1_CH9); no longer U1.19 (GPIO14/ADC2_CH3)
- net CAN_RX: now also U1.6 (GPIO1/ADC1_CH0)
- net CAN_TX: now also U1.7 (GPIO2/ADC1_CH1)
- net MISO: now also U1.18 (GPIO13/ADC2_CH2), U11.5 (SDO); no longer U1.16 (GPIO11/ADC2_CH0)
- net MOSI: now also U1.16 (GPIO11/ADC2_CH0), U11.3 (SDI); no longer U1.17 (GPIO12/ADC2_CH1)
- net SCLK: now also U1.17 (GPIO12/ADC2_CH1), U11.4 (SCK); no longer U1.18 (GPIO13/ADC2_CH2)
- net SD1_CS: now also U1.43 (GPIO38); no longer U1.9 (GPIO4/ADC1_CH3)
- net SD1_DET: now also U1.39 (GPIO34); no longer U1.15 (GPIO10/ADC1_CH9)
- net SS1: now also U1.12 (GPIO7/ADC1_CH6); no longer U1.10 (GPIO5/ADC1_CH4)
- net SS2: now also U1.13 (GPIO8/ADC1_CH7); no longer U1.11 (GPIO6/ADC1_CH5)
- net SS3: now also U1.14 (GPIO9/ADC1_CH8); no longer U1.12 (GPIO7/ADC1_CH6)
- net SS4: now also U1.11 (GPIO6/ADC1_CH5); no longer U1.13 (GPIO8/ADC1_CH7)
- net SS5: now also U1.10 (GPIO5/ADC1_CH4); no longer U1.14 (GPIO9/ADC1_CH8)
- net VSPI_MISO: now also U1.40 (GPIO35); no longer U1.43 (GPIO38)
- net VSPI_MOSI: now also U1.42 (GPIO37); no longer U1.41 (GPIO36)
- net VSPI_SCLK: now also U1.41 (GPIO36); no longer U1.42 (GPIO37)
- net +3V3 renamed +3.3V
- removed net HSPI_MISO: U1.40 (GPIO35), U11.5 (SDO)
- removed net HSPI_MOSI: U1.39 (GPIO34), U11.3 (SDI)
- net HSPI_SCLK: no longer names the net of U1.38 (GPIO33)
- net HSPI_SCLK: no longer U11.4 (SCK)
- no-connect marks 5 -> 23
Other:
- sheet USB -> UART ports: added none; removed 3.3V

Commit message: Review Changes Made (except for meme)
Connections:
- net RES: now reaches U1.36 (SPICLK_N/GPIO48)
- no-connect marks 23 -> 22
Other:
- sheet Pressure Sensors ports: added RES; removed none
Changed lines of the file:
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@@
   (no_connect (at 135.89 87.63))
   (no_connect (at 135.89 82.55))
-  (no_connect (at 135.89 115.57))
   (no_connect (at 69.85 77.47))
   (no_connect (at 135.89 128.27))
@@
     (stroke (width 0) (type default))
   )
+  (wire (pts (xy 227.33 53.34) (xy 228.6 53.34))
+    (stroke (width 0) (type default))
+  )
   (wire (pts (xy 68.58 102.87) (xy 69.85 102.87))
     (stroke (width 0) (type default))
@@
   )
   (wire (pts (xy 68.58 85.09) (xy 69.85 85.09))
+    (stroke (width 0) (type default))
+  )
+  (wire (pts (xy 138.43 115.57) (xy 135.89 115.57))
     (stroke (width 0) (type default))
   )
@@
     (effects (font (size 1.27 1.27)) (justify right bottom))
   )
+  (label "RES" (at 138.43 115.57 0) (fields_autoplaced)
+    (effects (font (size 1.27 1.27)) (justify left bottom))
+  )
   (label "MOSI" (at 149.86 46.99 180) (fields_autoplaced)
     (effects (font (size 1.27 1.27)) (justify right bottom))
@@
   )
   (label "RXD" (at 29.21 43.18 0) (fields_autoplaced)
+    (effects (font (size 1.27 1.27)) (justify left bottom))
+  )
+  (label "RES" (at 228.6 53.34 0) (fields_autoplaced)
     (effects (font (size 1.27 1.27)) (justify left bottom))
   )
@@
       (effects (font (size 1.27 1.27)) (justify left))
     )
-    (instances
+    (pin "RES" input (at 227.33 53.34 0)
+      (effects (font (size 1.27 1.27)) (justify right))
+    )
+    (instances

Commit message: artem review
Connections:
- net MOSI: now also U1.17 (GPIO12/ADC2_CH1); no longer U1.16 (GPIO11/ADC2_CH0)
- net SCLK: now also U1.16 (GPIO11/ADC2_CH0); no longer U1.17 (GPIO12/ADC2_CH1)
Changed lines of the file:
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@@
     (effects (font (size 1.27 1.27)) (justify left bottom))
   )
-  (label "MOSI" (at 68.58 97.79 180) (fields_autoplaced)
+  (label "MOSI" (at 68.58 100.33 180) (fields_autoplaced)
     (effects (font (size 1.27 1.27)) (justify right bottom))
   )
@@
     (effects (font (size 1.27 1.27)) (justify right bottom))
   )
-  (label "SCLK" (at 68.58 100.33 180) (fields_autoplaced)
+  (label "SCLK" (at 68.58 97.79 180) (fields_autoplaced)
     (effects (font (size 1.27 1.27)) (justify right bottom))
   )

Commit message: ordering
Parts:
- 12VLED1: value 12V_LED -> RED_LED
- 3V3LED1: value 3V3LED -> BLUE_LED
- C12: value 4.2pF -> DNP
- C13, C14: value C -> 11pF
- R5: value 47.5 -> DNP
- TXLED1: value TX_LED -> GREEN_LED
Changed lines of the file:
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@@
       (effects (font (size 1.27 1.27)))
     )
-    (property "Value" "TX_LED" (at 25.4 24.4856 0)
+    (property "Value" "GREEN_LED" (at 25.4 24.4856 0)
       (effects (font (size 1.27 1.27)))
     )
@@
       (effects (font (size 1.27 1.27)))
     )
-    (property "Value" "3V3LED" (at 54.61 18.6944 0)
+    (property "Value" "BLUE_LED" (at 54.61 18.6944 0)
       (effects (font (size 1.27 1.27)))
     )
@@
       (effects (font (size 1.27 1.27)))
     )
-    (property "Value" "12V_LED" (at 63.5 29.5656 0)
+    (property "Value" "RED_LED" (at 63.5 29.5656 0)
       (effects (font (size 1.27 1.27)))
     )
@@
       (effects (font (size 1.27 1.27)) (justify left))
     )
-    (property "Value" "C" (at 165.1 144.5514 90)
+    (property "Value" "11pF" (at 165.1 144.5514 90)
       (effects (font (size 1.27 1.27)) (justify left))
     )
@@
       (effects (font (size 1.27 1.27)) (justify left))
     )
-    (property "Value" "C" (at 163.83 124.2314 90)
+    (property "Value" "11pF" (at 163.83 124.2314 90)
       (effects (font (size 1.27 1.27)) (justify left))
     )
@@
       (effects (font (size 1.27 1.27)) (justify left))
     )
-    (property "Value" "4.2pF" (at 68.58 59.69 90)
+    (property "Value" "DNP" (at 68.58 59.69 90)
       (effects (font (size 1.27 1.27)) (justify left))
     )
@@
       (effects (font (size 1.27 1.27)))
     )
-    (property "Value" "47.5" (at 57.15 59.69 90)
-      (effects (font (size 1.27 1.27)))
-    )
+    (property "Value" "DNP" (at 57.15 59.69 90)
+      (effects (font (size 1.27 1.27)))
+    )
