File: Hardware/usb-uart.kicad_sch (KiCad schematic)
At the start: 8 parts, among them J2 USB_C_Receptacle_USB2.0

Commit message: ordering
Parts:
- R13: value 470 -> 5.1k
- USBLED1: value USB_LED -> WHITE_LED
Changed lines of the file:
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@@
       (effects (font (size 1.27 1.27)))
     )
-    (property "Value" "USB_LED" (at 162.56 89.8144 0)
+    (property "Value" "WHITE_LED" (at 162.56 89.8144 0)
       (effects (font (size 1.27 1.27)))
     )
@@
       (effects (font (size 1.27 1.27)))
     )
-    (property "Value" "470" (at 154.94 95.377 90)
+    (property "Value" "5.1k" (at 154.94 95.377 90)
       (effects (font (size 1.27 1.27)))
     )
